File: OpenUsbSerialAdapter.sch (KiCad schematic (older format))
At the start: 21 parts, among them J1 USB_A, J2 FTDI, SW1 SW_DPDT_x2, U1 MCP2200-I-SO, U2 AMS1117-3.3, Y1 12M

Commit message: PCB is routed
Parts:
- removed C4: CP1, Capacitor_Tantalum_SMD:CP_EIA-3216-18_Kemet-A_Pad1.58x1.35mm_HandSolder, symbol Device:CP1
- added C4: 100n, Capacitor_SMD:C_0805_2012Metric_Pad1.15x1.40mm_HandSolder, symbol Device:C
- C3: value 220u -> 330n; footprint Capacitor_SMD:C_1206_3216Metric_Pad1.42x1.75mm_HandSolder -> Capacitor_SMD:C_0805_2012Metric_Pad1.15x1.40mm_HandSolder
- SW1: footprint (none) -> Button_Switch_THT:SW_CuK_JS202011CQN_DPDT_Straight
Connections:
- net GND: now also C5.2, C6.2, C4.2
- net VCC: now also C4.1
Changed lines of the file:
@@
 Sheet 1 1
 Title "OpenUsbSerialAdapter"
-Date "2020-01-12"
+Date "2020-03-23"
 Rev "1git"
 Comp "SukkoPera"
-Comment1 ""
+Comment1 "Licensed under CERN OHL v.1.2"
 Comment2 ""
 Comment3 ""
@@
 P 7345 2500
 F 0 "C3" H 7460 2546 50  0000 L CNN
-F 1 "220u" H 7460 2455 50  0000 L CNN
-F 2 "Capacitor_SMD:C_1206_3216Metric_Pad1.42x1.75mm_HandSolder" H 7383 2350 50  0001 C CNN
+F 1 "330n" H 7460 2455 50  0000 L CNN
+F 2 "Capacitor_SMD:C_0805_2012Metric_Pad1.15x1.40mm_HandSolder" H 7383 2350 50  0001 C CNN
 F 3 "~" H 7345 2500 50  0001 C CNN
 	1    7345 2500
@@
 Wire Wire Line
 	2680 3030 2680 2930
-$Comp
-L power:+5V #PWR0103
-U 1 1 5E16C4F0
-P 2680 2930
-F 0 "#PWR0103" H 2680 2780 50  0001 C CNN
-F 1 "+5V" H 2695 3103 50  0000 C CNN
-F 2 "" H 2680 2930 50  0001 C CNN
-F 3 "" H 2680 2930 50  0001 C CNN
-	1    2680 2930
-	1    0    0    -1
-$EndComp
-$Comp
-L Device:CP1 C4
-U 1 1 5E16E2B3
-P 2680 3180
-F 0 "C4" H 2795 3226 50  0000 L CNN
-F 1 "CP1" H 2795 3135 50  0000 L CNN
-F 2 "Capacitor_Tantalum_SMD:CP_EIA-3216-18_Kemet-A_Pad1.58x1.35mm_HandSolder" H 2680 3180 50  0001 C CNN
-F 3 "~" H 2680 3180 50  0001 C CNN
-	1    2680 3180
-	1    0    0    -1
-$EndComp
 Wire Wire Line
 	2680 3330 2680 3415
@@
 	4425 5910 4425 6180
 Wire Wire Line
-	4425 6180 5480 6180
+	4425 6180 4950 6180
 Wire Wire Line
 	5480 6180 5480 5910
 Wire Wire Line
-	4950 5760 4950 6275
+	4950 5760 4950 6180
 $Comp
 L power:GND #PWR012
@@
 F 0 "SW1" H 6880 5675 50  0000 C CNN
 F 1 "SW_DPDT_x2" H 6880 5584 50  0000 C CNN
-F 2 "" H 6880 5390 50  0001 C CNN
+F 2 "Button_Switch_THT:SW_CuK_JS202011CQN_DPDT_Straight" H 6880 5390 50  0001 C CNN
 F 3 "~" H 6880 5390 50  0001 C CNN
 	1    6880 5390
@@
 F 0 "SW1" H 7025 1880 50  0000 C CNN
 F 1 "SW_DPDT_x2" H 7025 1971 50  0000 C CNN
-F 2 "" H 7025 2205 50  0001 C CNN
+F 2 "Button_Switch_THT:SW_CuK_JS202011CQN_DPDT_Straight" H 7025 2205 50  0001 C CNN
 F 3 "~" H 7025 2205 50  0001 C CNN
 	2    7025 2205
@@
 	1    0    0    -1
 $EndComp
+Connection ~ 4950 6180
+Wire Wire Line
+	4950 6180 5480 6180
+Wire Wire Line
+	4950 6180 4950 6275
+$Comp
+L power:VCC #PWR0103
+U 1 1 5EE1C505
+P 2680 2930
+F 0 "#PWR0103" H 2680 2780 50  0001 C CNN
+F 1 "VCC" H 2697 3103 50  0000 C CNN
+F 2 "" H 2680 2930 50  0001 C CNN
+F 3 "" H 2680 2930 50  0001 C CNN
+	1    2680 2930
+	1    0    0    -1
+$EndComp
+$Comp
+L Device:C C4
+U 1 1 5EE1F7D3
+P 2680 3180
+F 0 "C4" H 2795 3226 50  0000 L CNN
+F 1 "100n" H 2795 3135 50  0000 L CNN
+F 2 "Capacitor_SMD:C_0805_2012Metric_Pad1.15x1.40mm_HandSolder" H 2718 3030 50  0001 C CNN
+F 3 "~" H 2680 3180 50  0001 C CNN
+	1    2680 3180
+	1    0    0    -1
+$EndComp

Commit message: Done! (Again...)
Parts:
- C3: footprint Capacitor_SMD:C_0805_2012Metric_Pad1.15x1.40mm_HandSolder -> Capacitor_SMD:C_1206_3216Metric_Pad1.42x1.75mm_HandSolder
- J1: footprint Connector_USB:USB_A_Molex_105057_Vertical -> OpenUsbSerialAdapter:USB_A_Molex_48037
Changed lines of the file:
@@
 F 0 "J1" H 1637 3552 50  0000 C CNN
 F 1 "USB_A" H 1637 3461 50  0000 C CNN
-F 2 "Connector_USB:USB_A_Molex_105057_Vertical" H 1730 3035 50  0001 C CNN
+F 2 "OpenUsbSerialAdapter:USB_A_Molex_48037" H 1730 3035 50  0001 C CNN
 F 3 " ~" H 1730 3035 50  0001 C CNN
 	1    1580 3085
@@
 F 0 "C3" H 7460 2546 50  0000 L CNN
 F 1 "330n" H 7460 2455 50  0000 L CNN
-F 2 "Capacitor_SMD:C_0805_2012Metric_Pad1.15x1.40mm_HandSolder" H 7383 2350 50  0001 C CNN
+F 2 "Capacitor_SMD:C_1206_3216Metric_Pad1.42x1.75mm_HandSolder" H 7383 2350 50  0001 C CNN
 F 3 "~" H 7345 2500 50  0001 C CNN
 	1    7345 2500

Commit message: Some refinements
Parts:
- J2: footprint Connector_PinHeader_2.54mm:PinHeader_1x06_P2.54mm_Vertical -> OpenUsbSerialAdapter:PinHeader_1x06_P2.54mm_Vertical
Changed lines of the file:
@@
 F 0 "J2" H 9313 3051 50  0000 L CNN
 F 1 "FTDI" H 9313 2960 50  0000 L CNN
-F 2 "Connector_PinHeader_2.54mm:PinHeader_1x06_P2.54mm_Vertical" H 9285 3075 50  0001 C CNN
+F 2 "OpenUsbSerialAdapter:PinHeader_1x06_P2.54mm_Vertical" H 9285 3075 50  0001 C CNN
 F 3 "~" H 9285 3075 50  0001 C CNN
 	1    9285 3075

Commit message: Final touches
Parts:
- SW1: footprint Button_Switch_THT:SW_CuK_JS202011CQN_DPDT_Straight -> OpenUsbSerialAdapter:SW_DPDT
Changed lines of the file:
@@
 F 0 "SW1" H 6880 5675 50  0000 C CNN
 F 1 "SW_DPDT_x2" H 6880 5584 50  0000 C CNN
-F 2 "Button_Switch_THT:SW_CuK_JS202011CQN_DPDT_Straight" H 6880 5390 50  0001 C CNN
+F 2 "OpenUsbSerialAdapter:SW_DPDT" H 6880 5390 50  0001 C CNN
 F 3 "~" H 6880 5390 50  0001 C CNN
 	1    6880 5390
@@
 F 0 "SW1" H 7025 1880 50  0000 C CNN
 F 1 "SW_DPDT_x2" H 7025 1971 50  0000 C CNN
-F 2 "Button_Switch_THT:SW_CuK_JS202011CQN_DPDT_Straight" H 7025 2205 50  0001 C CNN
+F 2 "OpenUsbSerialAdapter:SW_DPDT" H 7025 2205 50  0001 C CNN
 F 3 "~" H 7025 2205 50  0001 C CNN
 	2    7025 2205

Commit message: Tune quartz tracks length
Connections:
- net clk+: now reaches C1.2, U1.2 (OSC1), Y1.1
- net clk-: now reaches C2.2, U1.3 (OSC2), Y1.2
Changed lines of the file:
@@
 	1    0    0    -1
 $EndComp
+Text Label 6850 3405 0    50   ~ 0
+clk+
+Text Label 6850 3875 0    50   ~ 0
+clk-
 $EndSCHEMATC
